Commit message: Fixed the peopeller direction problem

File: my_wamv/revised_urdf.urdf (robot description, URDF)
Before this commit: robot blueboat_urdf, 3 links, 2 joints
Joints:
- joint left_joint: axis -0.99648 0.083772 0 -> 0.99648 0.083772 0
- joint right_joint: axis -0.99648 0.083772 0 -> 0.99648 0.083772 0
